Commit message: Robot can take the box

File: arm_description/urdf/arm.urdf.xacro (robot description, xacro)
@@ -261,9 +261,28 @@
         </actuator>
     </transmission>
-    <link name="tool" />
-    <joint name="link_6-tool" type="fixed">
+    <link name="vacuum_gripper">
+        <gravity>0</gravity>
+        <visual>
+            <origin rpy="0 0 0" xyz="0 0 0" />
+            <geometry>
+                <box size="0.01 0.01 0.01" />
+            </geometry>
+            <material name="transparent">
+                <color rgba="0 0 0 0" />
+            </material>
+        </visual>
+        <inertial>
+            <origin rpy="0 0 0" xyz="0.000000 0.000000 0.000000" />
+            <mass value="0.0001" />
+            <inertia ixx="1e-08" ixy="0" ixz="0" iyy="1e-08" iyz="0" izz="1e-08" />
+        </inertial>
+    </link>
+    <joint name="gripper_joint" type="revolute">
+        <axis xyz="1 0 0" />
         <parent link="link_6" />
-        <child link="tool" />
+        <child link="vacuum_gripper" />
         <origin xyz="0 0 0" rpy="0 ${DEG2RAD * 90} 0" />
+        <limit effort="50" velocity="50" lower="0" upper="0" />
+        <dynamics damping="0.0" friction="10" />
     </joint>
     <!-- Controllers -->
@@ -274,3 +293,11 @@
         </plugin>
     </gazebo>
+    <!-- Gripper -->
+    <gazebo>
+        <plugin name="gazebo_ros_vacuum_gripper" filename="libgazebo_ros_vacuum_gripper.so">
+            <robotNamespace>/kuka_arm/vacuum_gripper</robotNamespace>
+            <bodyName>vacuum_gripper</bodyName>
+            <topicName>grasping</topicName>
+        </plugin>
+    </gazebo>
 </robot>
